File: PCB/WildfireDetectionSystem.brd (EAGLE design)
At the start: 80 x 60 mm, 95 parts, among them IC1 STM32L476RGT6, J1 10118192-0001LF, J3 B4B-XH-A, J4 B5B-XH-A, J7 B4B-PH-K-S, J8 U.FL-R-SMT-1(10), J9 B2B-PH-K-S, SW1 434133025816, U1 BME280, U3 NEO-6M-GPS, U4 TPS62142RGTT, U5 TPS61022RWUR, U6 LMR33630ADDA, U7 BQ24074RGTR, Y1 ABLS-8.000MHZ-B2-T, Y2 ECS-.327-12.5-12QS-TR

Commit message: pcbv2
Parts:
- added L2: L_1R0_0805, JLC PCB Basic Parts_loc:R0805
- moved D9 1.30 mm to (32.4, -2.50)
Connections:
- new net N$16: L2.2, L6.2
- net SW3: now also L2.1; no longer L6.2
Routing:
- net 5V_IN: track 64.7 -> 69.2 mm
- net N$16: track 0.00 -> 2.64 mm
- net SW3: track 8.47 -> 10.3 mm
- net 5V_IN_SOLAR: track 17.4 -> 16.1 mm
Changed lines of the file:
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@@
 <attribute name="SNAPEDA_LINK" value="https://www.snapeda.com/parts/SS34LWH/taiwan/view-part/?ref=snap" x="8.9" y="-0.8" size="1.778" layer="27" rot="R180" display="off"/>
 </element>
-<element name="D9" library="SS34LWH" package="SODFL3718X102N" value="SS34LWH" x="31.1" y="-2.4" smashed="yes">
-<attribute name="AVAILABILITY" value="In Stock" x="31.1" y="-2.4" size="1.778" layer="27" display="off"/>
-<attribute name="CHECK_PRICES" value="https://www.snapeda.com/parts/SS34LWH/taiwan/view-part/?ref=eda" x="31.1" y="-2.4" size="1.778" layer="27" display="off"/>
-<attribute name="DESCRIPTION" value="                                                      3A, 40V, Automotive Planar Schottky                                              " x="31.1" y="-2.4" size="1.778" layer="27" display="off"/>
-<attribute name="MF" value="Taiwan Semiconductor" x="31.1" y="-2.4" size="1.778" layer="27" display="off"/>
-<attribute name="MP" value="SS34LWH" x="31.1" y="-2.4" size="1.778" layer="27" display="off"/>
-<attribute name="PACKAGE" value="SOD-123W-2 Taiwan Semiconductor" x="31.1" y="-2.4" size="1.778" layer="27" display="off"/>
-<attribute name="PRICE" value="None" x="31.1" y="-2.4" size="1.778" layer="27" display="off"/>
-<attribute name="SNAPEDA_LINK" value="https://www.snapeda.com/parts/SS34LWH/taiwan/view-part/?ref=snap" x="31.1" y="-2.4" size="1.778" layer="27" display="off"/>
+<element name="D9" library="SS34LWH" package="SODFL3718X102N" value="SS34LWH" x="32.4" y="-2.5" smashed="yes">
+<attribute name="AVAILABILITY" value="In Stock" x="32.4" y="-2.5" size="1.778" layer="27" display="off"/>
+<attribute name="CHECK_PRICES" value="https://www.snapeda.com/parts/SS34LWH/taiwan/view-part/?ref=eda" x="32.4" y="-2.5" size="1.778" layer="27" display="off"/>
+<attribute name="DESCRIPTION" value="                                                      3A, 40V, Automotive Planar Schottky                                              " x="32.4" y="-2.5" size="1.778" layer="27" display="off"/>
+<attribute name="MF" value="Taiwan Semiconductor" x="32.4" y="-2.5" size="1.778" layer="27" display="off"/>
+<attribute name="MP" value="SS34LWH" x="32.4" y="-2.5" size="1.778" layer="27" display="off"/>
+<attribute name="PACKAGE" value="SOD-123W-2 Taiwan Semiconductor" x="32.4" y="-2.5" size="1.778" layer="27" display="off"/>
+<attribute name="PRICE" value="None" x="32.4" y="-2.5" size="1.778" layer="27" display="off"/>
+<attribute name="SNAPEDA_LINK" value="https://www.snapeda.com/parts/SS34LWH/taiwan/view-part/?ref=snap" x="32.4" y="-2.5" size="1.778" layer="27" display="off"/>
 </element>
 <element name="D10" library="SS34LWH" package="SODFL3718X102N" value="SS34LWH" x="8.2" y="9.4" smashed="yes" rot="R90">
@@
 <attribute name="LCSC_STOCK" value="37908" x="24.9" y="-2.1" size="1.778" layer="27" display="off"/>
 <attribute name="PROPERTIES" value="ManuPN: CMI201209U2R2KT 50mA 2.2uH ±10% 600mOhm 0805  ROHS" x="24.9" y="-2.1" size="1.778" layer="27" display="off"/>
+</element>
+<element name="L2" library="JLC PCB Basic Parts_loc" package="R0805" package3d_urn="urn:adsk.eagle:package:23553/2" value="L_1R0_0805" x="28.1" y="-2.1" smashed="yes" rot="R270">
+<attribute name="LCSC_DATASHEET" value="https://datasheet.lcsc.com/lcsc/2110081230_Sunlord-SDFL2012Q1R0KTF_C1042.pdf" x="28.1" y="-2.1" size="1.778" layer="27" rot="R270" display="off"/>
+<attribute name="LCSC_PART" value="C1042" x="28.1" y="-2.1" size="1.778" layer="27" rot="R270" display="off"/>
+<attribute name="LCSC_PRICE1_EUR" value="" x="28.1" y="-2.1" size="1.778" layer="27" rot="R270" display="off"/>
+<attribute name="LCSC_ROTATION_CCW" value="0" x="28.1" y="-2.1" size="1.778" layer="27" rot="R270" display="off"/>
+<attribute name="LCSC_STOCK" value="44995" x="28.1" y="-2.1" size="1.778" layer="27" rot="R270" display="off"/>
+<attribute name="PROPERTIES" value="ManuPN: SDFL2012Q1R0KTF 50mA 1uH ±10% 400mOhm 0805  ROHS" x="28.1" y="-2.1" size="1.778" layer="27" rot="R270" display="off"/>
 </element>
 </elements>
@@
 <wire x1="32" y1="-4.75" x2="29.8" y2="-4.75" width="0.2032" layer="1"/>
 <wire x1="29.8" y1="-4.75" x2="27.6" y2="-4.75" width="0.2032" layer="1"/>
-<wire x1="27.6" y1="-4.75" x2="27.6" y2="-4.4" width="0.2032" layer="1"/>
-<wire x1="27.6" y1="-4.4" x2="26.9" y2="-3.7" width="0.2032" layer="1"/>
-<via x="26.9" y="-3.7" extent="1-16" drill="0.35"/>
+<wire x1="27.6" y1="-4.75" x2="27.35" y2="-4.75" width="0.2032" layer="1"/>
+<wire x1="27.35" y1="-4.75" x2="26.7" y2="-4.1" width="0.2032" layer="1"/>
+<wire x1="26.7" y1="-4.1" x2="26.7" y2="-4" width="0.2032" layer="1"/>
+<via x="26.7" y="-4" extent="1-16" drill="0.35"/>
 <wire x1="7.765" y1="-11.05" x2="7.365" y2="-11.45" width="0.2032" layer="1"/>
 <wire x1="7.365" y1="-11.45" x2="7.365" y2="-12.835" width="0.2032" layer="1"/>
@@
 <wire x1="8.1" y1="2.7" x2="8.1" y2="5.6" width="0.3048" layer="1"/>
 <wire x1="8.1" y1="2.7" x2="9.5" y2="1.3" width="0.3048" layer="1"/>
-<wire x1="21.7" y1="0" x2="26.3" y2="0" width="0.3048" layer="1"/>
+<wire x1="21.5" y1="0.2" x2="29.8" y2="0.2" width="0.3048" layer="1"/>
 <wire x1="9.5" y1="1.3" x2="20.4" y2="1.3" width="0.3048" layer="1"/>
-<wire x1="20.4" y1="1.3" x2="21.7" y2="0" width="0.3048" layer="1"/>
+<wire x1="20.4" y1="1.3" x2="21.5" y2="0.2" width="0.3048" layer="1"/>
 <wire x1="10.65" y1="-8.165" x2="10.65" y2="-6.6" width="0.3048" layer="1"/>
 <wire x1="10.65" y1="-6.6" x2="14.3407875" y2="-6.6" width="0.3048" layer="1"/>
@@
 <wire x1="14.3407875" y1="-6.6" x2="14.6447875" y2="-6.904" width="0.3048" layer="1"/>
 <wire x1="14.6447875" y1="-6.904" x2="16.904" y2="-6.904" width="0.3048" layer="1"/>
-<wire x1="18.1" y1="-8.1" x2="20.6" y2="-8.1" width="0.3048" layer="1"/>
-<wire x1="20.6" y1="-8.1" x2="21.1" y2="-8.1" width="0.3048" layer="1"/>
+<wire x1="18.1" y1="-8.1" x2="21.1" y2="-8.1" width="0.3048" layer="1"/>
 <wire x1="9.95" y1="-8.865" x2="10.65" y2="-8.165" width="0.254" layer="1"/>
 <contactref element="D10" pad="C"/>
@@
 <wire x1="8.976" y1="6.476" x2="8.2" y2="7.252" width="0.3048" layer="1"/>
 <wire x1="8.2" y1="7.252" x2="8.2" y2="7.825" width="0.3048" layer="1"/>
-<wire x1="29.525" y1="-2.4" x2="28.7" y2="-2.4" width="0.3048" layer="1"/>
-<wire x1="28.7" y1="-2.4" x2="26.3" y2="0" width="0.3048" layer="1"/>
-<wire x1="28.7" y1="-2.4" x2="27.2" y2="-2.4" width="0.3048" layer="1"/>
-<via x="27.2" y="-2.4" extent="1-16" drill="0.35"/>
-<wire x1="27.2" y1="-2.4" x2="21.5" y2="-8.1" width="0.3048" layer="16"/>
-<wire x1="21.5" y1="-8.1" x2="21.1" y2="-8.1" width="0.3048" layer="16"/>
+<via x="29.6" y="-3.5" extent="1-16" drill="0.35"/>
+<wire x1="29.6" y1="-3.5" x2="25" y2="-8.1" width="0.3048" layer="16"/>
+<wire x1="25" y1="-8.1" x2="21.1" y2="-8.1" width="0.3048" layer="16"/>
 <via x="21.1" y="-8.1" extent="1-16" drill="0.35"/>
 <wire x1="21.1" y1="-8.1" x2="20.6" y2="-8.1" width="0.3048" layer="16"/>
@@
 <wire x1="15.9" y1="-12.8" x2="14.95" y2="-13.75" width="0.3048" layer="1"/>
 <wire x1="14.95" y1="-13.75" x2="14.6" y2="-13.75" width="0.3048" layer="1"/>
+<wire x1="30.6" y1="-2.5" x2="30.825" y2="-2.5" width="0.3048" layer="1"/>
+<wire x1="29.6" y1="-3.5" x2="30.6" y2="-2.5" width="0.3048" layer="1"/>
+<wire x1="29.8" y1="0.2" x2="30.825" y2="-0.825" width="0.3048" layer="1"/>
+<wire x1="30.825" y1="-0.825" x2="30.825" y2="-2.5" width="0.3048" layer="1"/>
 </signal>
 <signal name="PC14-OSC32-IN">
@@
 <wire x1="18.5" y1="-0.195" x2="21.045" y2="-0.195" width="0.3048" layer="1"/>
 <wire x1="21.045" y1="-0.195" x2="22.15" y2="-1.3" width="0.3048" layer="1"/>
-<contactref element="L6" pad="2"/>
-<wire x1="25.85" y1="-2.1" x2="24.65" y2="-0.9" width="0.3048" layer="1"/>
-<wire x1="22.55" y1="-0.9" x2="22.15" y2="-1.3" width="0.3048" layer="1"/>
-<wire x1="24.65" y1="-0.9" x2="22.55" y2="-0.9" width="0.3048" layer="1"/>
+<wire x1="22.15" y1="-1.3" x2="22.55" y2="-0.9" width="0.3048" layer="1"/>
+<contactref element="L2" pad="1"/>
+<wire x1="27.85" y1="-0.9" x2="28.1" y2="-1.15" width="0.3048" layer="1"/>
+<wire x1="22.55" y1="-0.9" x2="27.85" y2="-0.9" width="0.3048" layer="1"/>
 </signal>
 <signal name="N$15">
@@
 <wire x1="34.2" y1="-6.45" x2="35.1" y2="-5.55" width="0.3048" layer="1"/>
 <wire x1="35.1" y1="-5.55" x2="35.1" y2="-2.9" width="0.3048" layer="1"/>
-<wire x1="35.1" y1="-2.9" x2="34.6" y2="-2.4" width="0.3048" layer="1"/>
-<wire x1="34.6" y1="-2.4" x2="32.675" y2="-2.4" width="0.3048" layer="1"/>
+<wire x1="35.1" y1="-2.9" x2="34.7" y2="-2.5" width="0.3048" layer="1"/>
+<wire x1="34.7" y1="-2.5" x2="33.975" y2="-2.5" width="0.3048" layer="1"/>
 <contactref element="L5" pad="1"/>
 <wire x1="25.55" y1="-6.5" x2="25.55" y2="-4.3" width="0.3048" layer="1"/>
@@
 <wire x1="23.95" y1="-4.2" x2="23.85" y2="-4.3" width="0.3048" layer="1"/>
 </signal>
+<signal name="N$16">
+<contactref element="L6" pad="2"/>
+<contactref element="L2" pad="2"/>
+<wire x1="28.1" y1="-3.05" x2="26.8" y2="-3.05" width="0.3048" layer="1"/>
+<wire x1="26.8" y1="-3.05" x2="25.85" y2="-2.1" width="0.3048" layer="1"/>
+</signal>
 </signals>

Commit message: pcbv2
Parts:
- added C23, C39: C_10UF/25V_0805, JLC PCB Basic Parts_loc:C0805
- added C4, C5: C_10UF/10V_0603, JLC PCB Basic Parts_loc:C0603
- added C40, C41, C42: C_22UF/25V_0805, JLC PCB Basic Parts_loc:C0805
- added C43: C_100NF/50V_0603, JLC PCB Basic Parts_loc:C0603
- added L8: L_1R0_0805, JLC PCB Basic Parts_loc:R0805
- added R24: R_100K_0603, JLC PCB Basic Parts_loc:R0603
- added R25: R_680K_0603, JLC PCB Basic Parts_loc:R0603
- added R26: R_130K_0603, JLC PCB Basic Parts_loc:R0603
- added R6: R_10K_0603, JLC PCB Basic Parts_loc:R0603
- added U2: TPS63070RNMR, TPS63070RNMR:VREG_TPS63070RNMR
- moved C24 16.3 mm to (25.2, 21.6), turned to 180 degrees
- moved C25 15.3 mm to (25.2, 19.9), turned to 180 degrees
- moved Y2 11.6 mm to (28.6, 20.7), turned to 90 degrees
- moved C9 7.98 mm to (26.4, 15.2), turned to 270 degrees
- moved C38 7.47 mm to (22.2, -14.3)
- moved C19 7.34 mm to (26.0, 11.9)
- moved C10 6.85 mm to (23.6, 14.9), turned to 270 degrees
- moved C6 6.74 mm to (30.4, 15.2), turned to 270 degrees
- moved C37 6.45 mm to (23.5, -17.1)
- moved C36 6.26 mm to (27.2, -17.1)
- moved R11 6.18 mm to (37.9, 22.2), turned to 90 degrees
- moved U4 6.17 mm to (25.1, -14.2)
- moved C11 6.16 mm to (27.7, 15.2), turned to 270 degrees
- moved R22 6.16 mm to (28.8, -12.6)
- moved SW1 6.02 mm to (19.6, 15.3), turned to 270 degrees
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Connections:
- new net 5V_BUCK: C16.1, C4.2, C40.1, C41.1, C42.1, R24.2, R25.1, U2.7_8, U7.13
- new net N$19: L8.1, U2.11
- new net N$20: L8.2, U2.9
- new net N$21: R6.1, U2.1, U2.14
- new net N$22: R24.1, U2.2
- new net N$23: R25.2, R26.2, U2.5
- new net VAUX: C43.1, U2.3
- net 5V_IN: now also C23.1, C39.1, C5.2, R6.2, U2.12_13; no longer C16.1, U7.13
- net GND: now also C23.2, C39.2, C4.1, C40.2, C41.2, C42.2, C43.2, C5.1, R26.1, U2.10, U2.15, U2.4, U2.6
Routing:
- net I2C1_SCL_BME: track 65.8 -> 38.6 mm
- net 5V_BUCK: track 0.00 -> 24.9 mm
- net GND: track 198.9 -> 222.0 mm, vias 53 -> 55
- net I2C1_SDA_BME: track 51.0 -> 35.9 mm
- net N$22: track 0.00 -> 15.0 mm, vias 0 -> 2
- net 5V_IN: track 69.2 -> 79.6 mm
- net PC14-OSC32-IN: track 8.88 -> 17.1 mm
- net PC15-OSC32-OUT: track 9.72 -> 16.8 mm
- net UART3_RX_GPS: track 113.5 -> 106.5 mm
- net N$23: track 0.00 -> 6.13 mm
- net NRST: track 73.0 -> 67.0 mm
- net N$21: track 0.00 -> 4.67 mm
- net UART1_RX_LORA: track 68.1 -> 64.0 mm, vias 2 -> 1
- net UART1_TX_LORA: track 68.8 -> 65.0 mm, vias 4 -> 2
- net 3V3: track 63.9 -> 60.0 mm, vias 19 -> 17
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