File: PCB/WildfireDetectionSystem.sch (EAGLE design)
At the start: 99 parts, among them IC1 STM32L476RGT6, J1 10118192-0001LF, J3 B4B-XH-A, J4 B5B-XH-A, J5 B2B-PH-K-S, J7 B4B-PH-K-S, J8 U.FL-R-SMT-1(10), SW1 434133025816, U1 BME280, U2 TPS63070RNMT, U3 NEO-6M-GPS, U4 TPS62142RGTT, U5 TPS61022RWUR, U7 BQ24074RGTR, Y1 ABLS-8.000MHZ-B2-T, Y2 ECS-.327-12.5-12QS-TR

Commit message: pcbv2
Parts:
- D10, D9: value SS34LWH -> DSK34; device SS34LWH:SS34LWH -> MDD_DSK34_LCSC_C41029:DSK34
- U$1: value 24LC32AT-I/SN -> 24LC32AT-I_SN; device 24LC32AT-I_SN:24LC32AT-I/SN -> MICROCHIP_24LC32AT-I_SN_LCSC_C615715:24LC32AT-I_SN
Other:
- moved on the sheet: D10, D9
Changed lines of the file:
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@@
 <part name="J4" library="B5B-XH-A" library_urn="urn:adsk.eagle:library:52044919" deviceset="B5B-XH-A" device="" package3d_urn="urn:adsk.eagle:package:52044922/2"/>
 <part name="D5" library="ce-capstone" library_urn="urn:adsk.eagle:library:52044969" deviceset="SML-P12MTT86" device="" package3d_urn="urn:adsk.eagle:package:52045011/1"/>
-<part name="U$1" library="24LC32AT-I_SN" library_urn="urn:adsk.eagle:library:52044924" deviceset="24LC32AT-I/SN" device="" package3d_urn="urn:adsk.eagle:package:52044927/1"/>
+<part name="U$1" library="MICROCHIP_24LC32AT-I_SN_LCSC_C615715" deviceset="24LC32AT-I_SN" device=""/>
 <part name="C1" library="CL05B104KO5NNNC" library_urn="urn:adsk.eagle:library:52044934" deviceset="CL05B104KO5NNNC" device="" package3d_urn="urn:adsk.eagle:package:52044937/2"/>
 <part name="C2" library="CL10C200JB8NNNC" library_urn="urn:adsk.eagle:library:52044939" deviceset="CL10C200JB8NNNC" device="" package3d_urn="urn:adsk.eagle:package:52044942/2"/>
@@
 <part name="C38" library="JLC PCB Basic Parts_loc" deviceset="C_" device="_0603" package3d_urn="urn:adsk.eagle:package:23616/2" technology="3.3NF/50V" value="3.3nF"/>
 <part name="U$5" library="NC_MARKER" deviceset="NC_MARKER" device=""/>
-<part name="D9" library="SS34LWH" deviceset="SS34LWH" device=""/>
-<part name="D10" library="SS34LWH" deviceset="SS34LWH" device=""/>
+<part name="D9" library="MDD_DSK34_LCSC_C41029" deviceset="DSK34" device=""/>
+<part name="D10" library="MDD_DSK34_LCSC_C41029" deviceset="DSK34" device=""/>
 <part name="R23" library="JLC PCB Basic Parts_loc" deviceset="R_" device="_0603" package3d_urn="urn:adsk.eagle:package:23555/3" technology="10K" value="10k"/>
 <part name="C3" library="JLC PCB Basic Parts_loc" deviceset="C_" device="_0603" package3d_urn="urn:adsk.eagle:package:23616/2" technology="22UF/6.3V" value="22uF"/>
@@
 <attribute name="NAME" x="233.172" y="-29.464" size="1.778" layer="95" rot="R180"/>
 </instance>
-<instance part="U$1" gate="A" x="162.56" y="20.32" smashed="yes">
-<attribute name="NAME" x="157.22028125" y="35.2204" size="2.08503125" layer="95" ratio="10" rot="SR0"/>
-<attribute name="VALUE" x="156.07388125" y="-2.7502" size="2.08573125" layer="96" ratio="10" rot="SR0"/>
+<instance part="U$1" gate="G$1" x="160.02" y="20.32" smashed="yes">
+<attribute name="NAME" x="154.68028125" y="35.2204" size="2.08503125" layer="95" ratio="10" rot="SR0"/>
+<attribute name="VALUE" x="153.53388125" y="-2.7502" size="2.08573125" layer="96" ratio="10" rot="SR0"/>
 </instance>
 <instance part="C1" gate="G$1" x="203.2" y="106.68" smashed="yes" rot="R270">
@@
 </instance>
 <instance part="U$5" gate="G$1" x="381" y="-10.16" smashed="yes" rot="R180"/>
-<instance part="D9" gate="G$1" x="424.18" y="121.92" smashed="yes">
-<attribute name="NAME" x="419.1" y="124.46" size="1.778" layer="95"/>
-<attribute name="VALUE" x="419.1" y="118.11" size="1.778" layer="96"/>
-</instance>
-<instance part="D10" gate="G$1" x="200.66" y="78.74" smashed="yes" rot="R180">
-<attribute name="NAME" x="200.66" y="76.2" size="1.778" layer="95" rot="R180"/>
-<attribute name="VALUE" x="203.2" y="85.09" size="1.778" layer="96" rot="R180"/>
+<instance part="D9" gate="G$1" x="424.18" y="121.92" smashed="yes" rot="R180">
+<attribute name="NAME" x="429.26" y="119.38" size="1.778" layer="95" rot="R180"/>
+<attribute name="VALUE" x="429.26" y="125.73" size="1.778" layer="96" rot="R180"/>
+</instance>
+<instance part="D10" gate="G$1" x="200.66" y="78.74" smashed="yes">
+<attribute name="NAME" x="200.66" y="81.28" size="1.778" layer="95"/>
+<attribute name="VALUE" x="198.12" y="72.39" size="1.778" layer="96"/>
 </instance>
 <instance part="R23" gate="R1" x="322.58" y="7.62" smashed="yes">
@@
 </segment>
 <segment>
-<pinref part="U$1" gate="A" pin="VCC"/>
-<wire x1="144.78" y1="27.94" x2="132.08" y2="27.94" width="0.1524" layer="91"/>
-<label x="134.62" y="27.94" size="1.778" layer="95"/>
+<pinref part="U$1" gate="G$1" pin="VCC"/>
+<label x="180.34" y="22.86" size="1.778" layer="95"/>
+<wire x1="168.91" y1="24.0792" x2="180.34" y2="24.0792" width="0.1524" layer="91"/>
 </segment>
 <segment>
@@
 </segment>
 <segment>
-<pinref part="U$1" gate="A" pin="VSS"/>
-<wire x1="144.78" y1="5.08" x2="132.08" y2="5.08" width="0.1524" layer="91"/>
-<label x="134.62" y="5.08" size="1.778" layer="95"/>
-</segment>
-<segment>
-<pinref part="U$1" gate="A" pin="WP"/>
-<pinref part="U$1" gate="A" pin="A0"/>
-<wire x1="144.78" y1="20.32" x2="144.78" y2="15.24" width="0.1524" layer="91"/>
-<pinref part="U$1" gate="A" pin="A1"/>
-<wire x1="144.78" y1="15.24" x2="144.78" y2="12.7" width="0.1524" layer="91"/>
-<junction x="144.78" y="15.24"/>
-<pinref part="U$1" gate="A" pin="A2"/>
-<wire x1="144.78" y1="12.7" x2="144.78" y2="10.16" width="0.1524" layer="91"/>
-<junction x="144.78" y="12.7"/>
-<wire x1="144.78" y1="12.7" x2="137.16" y2="12.7" width="0.1524" layer="91"/>
-<label x="137.16" y="12.7" size="1.778" layer="95"/>
+<pinref part="U$1" gate="G$1" pin="VSS"/>
+<label x="137.16" y="15.24" size="1.778" layer="95"/>
+<wire x1="151.13" y1="16.4592" x2="137.16" y2="16.4592" width="0.1524" layer="91"/>
+</segment>
+<segment>
+<pinref part="U$1" gate="G$1" pin="A0"/>
+<pinref part="U$1" gate="G$1" pin="A1"/>
+<wire x1="151.13" y1="24.0792" x2="151.13" y2="21.5392" width="0.1524" layer="91"/>
+<pinref part="U$1" gate="G$1" pin="A2"/>
+<wire x1="151.13" y1="21.5392" x2="151.13" y2="18.9992" width="0.1524" layer="91"/>
+<junction x="151.13" y="21.5392"/>
+<label x="137.16" y="22.86" size="1.778" layer="95"/>
+<wire x1="151.13" y1="21.5392" x2="137.16" y2="21.5392" width="0.1524" layer="91"/>
 </segment>
 <segment>
@@
 <wire x1="383.54" y1="104.14" x2="391.16" y2="104.14" width="0.1524" layer="91"/>
 <label x="386.08" y="104.14" size="1.778" layer="95"/>
+</segment>
+<segment>
+<pinref part="U$1" gate="G$1" pin="WP"/>
+<wire x1="168.91" y1="21.5392" x2="180.34" y2="21.5392" width="0.1524" layer="91"/>
+<label x="180.34" y="20.32" size="1.778" layer="95"/>
 </segment>
 </net>
@@
 <segment>
 <pinref part="D10" gate="G$1" pin="K"/>
-<wire x1="195.58" y1="78.74" x2="187.96" y2="78.74" width="0.1524" layer="91"/>
+<wire x1="195.58" y1="78.867" x2="187.96" y2="78.74" width="0.1524" layer="91"/>
 <label x="187.96" y="78.74" size="1.778" layer="95"/>
 </segment>
@@
 <segment>
 <pinref part="D9" gate="G$1" pin="K"/>
-<wire x1="429.26" y1="121.92" x2="429.26" y2="129.54" width="0.1524" layer="91"/>
+<wire x1="429.26" y1="121.793" x2="429.26" y2="129.54" width="0.1524" layer="91"/>
 <label x="426.72" y="129.54" size="1.778" layer="95"/>
 </segment>
@@
 </segment>
 <segment>
-<pinref part="U$1" gate="A" pin="SCL"/>
-<wire x1="144.78" y1="22.86" x2="132.08" y2="22.86" width="0.1524" layer="91"/>
-<label x="134.62" y="22.86" size="1.778" layer="95"/>
+<pinref part="U$1" gate="G$1" pin="SCL"/>
+<label x="180.34" y="17.78" size="1.778" layer="95"/>
+<wire x1="168.91" y1="18.9992" x2="180.34" y2="18.9992" width="0.1524" layer="91"/>
 </segment>
 </net>
@@
 </segment>
 <segment>
-<pinref part="U$1" gate="A" pin="SDA"/>
-<wire x1="180.34" y1="27.94" x2="195.58" y2="27.94" width="0.1524" layer="91"/>
-<label x="182.88" y="27.94" size="1.778" layer="95"/>
+<pinref part="U$1" gate="G$1" pin="SDA"/>
+<label x="180.34" y="15.24" size="1.778" layer="95"/>
+<wire x1="168.91" y1="16.4592" x2="180.34" y2="16.4592" width="0.1524" layer="91"/>
 </segment>
 </net>
@@
 <segment>
 <pinref part="J1" gate="G$1" pin="VUSB"/>
-<wire x1="218.44" y1="78.74" x2="205.74" y2="78.74" width="0.1524" layer="91"/>
+<wire x1="218.44" y1="78.74" x2="205.74" y2="78.867" width="0.1524" layer="91"/>
 <label x="205.74" y="78.74" size="1.778" layer="95"/>
 <pinref part="D10" gate="G$1" pin="A"/>
-<junction x="205.74" y="78.74"/>
+<junction x="205.74" y="78.867"/>
 </segment>
 </net>
@@
 <wire x1="406.4" y1="121.92" x2="411.48" y2="121.92" width="0.1524" layer="91"/>
 <junction x="406.4" y="121.92"/>
-<wire x1="411.48" y1="121.92" x2="419.1" y2="121.92" width="0.1524" layer="91"/>
+<wire x1="411.48" y1="121.92" x2="419.1" y2="121.793" width="0.1524" layer="91"/>
 <junction x="411.48" y="121.92"/>
 <pinref part="R24" gate="R1" pin="2"/>
